File: hardware/SDCard.kicad_sch (KiCad schematic)
At the start: 12 parts, among them J5 Micro_SD_Card_Det_Hirose_DM3AT, U6 PCF8563TS, Y3 X321532768KGD2SI

Commit message: fix: unavailable components
Parts:
- J5: footprint AuraMon:MOLEX_104031-0811 -> AuraMon:AMPHENOL_1140084168; JLCPCB Part # C585350 -> C3195424; MPN 1040310811 -> 114-00841-68; Manufacturer MOLEX -> Amphenol ICC
Changed lines of the file:
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@@
 			)
 		)
-		(property "Footprint" "AuraMon:MOLEX_104031-0811"
+		(property "Footprint" "AuraMon:AMPHENOL_1140084168"
 			(at 153.67 77.47 0)
 			(effects
@@
 			)
 		)
-		(property "Datasheet" "https://www.molex.com/content/dam/molex/molex-dot-com/products/automated/en-us/salesdrawingpdf/104/104031/1040310811_sd.pdf?inline"
+		(property "Datasheet" "https://jlcpcb.com/api/file/downloadByFileSystemAccessId/8589834893502427136"
 			(at 101.6 92.71 0)
 			(effects
@@
 			)
 		)
-		(property "Description" "-25℃~+85℃ 1.42mm Connector and Ejector MicroSD Card (TF Card) Push-Pull SMD SD Card / Memory Card Connector ROHS"
+		(property "Description" "1.55mm Connector and Ejector MicroSD Card (TF Card) No Push-Pull SMD SD Card / Memory Card Connector ROHS"
 			(at 101.6 95.25 0)
 			(effects
@@
 			)
 		)
-		(property "MPN" "1040310811"
+		(property "MPN" " 114-00841-68"
 			(at 101.6 95.25 0)
 			(effects
@@
 			)
 		)
-		(property "Manufacturer" "MOLEX"
+		(property "Manufacturer" "Amphenol ICC"
 			(at 101.6 95.25 0)
 			(effects
@@
 			)
 		)
-		(property "JLCPCB Part #" "C585350"
+		(property "JLCPCB Part #" " C3195424"
 			(at 101.6 95.25 0)
 			(effects
